Commit message: Fix motor direction and URDF configuration for rasptank differential drive

File: rasptank_diff_drive/description/urdf/diffbot.urdf.xacro (robot description, xacro)
@@ -4,9 +4,91 @@
   <xacro:arg name="prefix" default="" />
   <xacro:arg name="use_mock_hardware" default="false" />
-  <xacro:include filename="$(find ros2_control_demo_description)/diffbot/urdf/diffbot_description.urdf.xacro" />
-  <!-- Import Rviz colors -->
-  <xacro:include filename="$(find ros2_control_demo_description)/diffbot/urdf/diffbot.materials.xacro" />
   <!-- Import diffbot ros2_control description -->
-  <xacro:include filename="$(find rasptank_diff_drive)/ros2_control/diffbot.ros2_control.xacro" />
+  <xacro:include filename="../ros2_control/diffbot_ros2_control.xacro" />
+  <!-- Robot physical description -->
+  <xacro:macro name="diffbot" params="prefix">
+    <link name="${prefix}base_link">
+      <visual>
+        <origin xyz="0 0 0.1" rpy="0 0 0"/>
+        <geometry>
+          <box size="0.4 0.3 0.2"/>
+        </geometry>
+        <material name="blue">
+          <color rgba="0 0 1 1"/>
+        </material>
+      </visual>
+      <collision>
+        <origin xyz="0 0 0.1" rpy="0 0 0"/>
+        <geometry>
+          <box size="0.4 0.3 0.2"/>
+        </geometry>
+      </collision>
+      <inertial>
+        <origin xyz="0 0 0.1" rpy="0 0 0"/>
+        <mass value="5.0"/>
+        <inertia ixx="0.08" ixy="0.0" ixz="0.0" iyy="0.13" iyz="0.0" izz="0.2"/>
+      </inertial>
+    </link>
+    <!-- Left wheel -->
+    <link name="${prefix}left_wheel">
+      <visual>
+        <origin xyz="0 0 0" rpy="1.5708 0 0"/>
+        <geometry>
+          <cylinder radius="0.1" length="0.05"/>
+        </geometry>
+        <material name="black">
+          <color rgba="0 0 0 1"/>
+        </material>
+      </visual>
+      <collision>
+        <origin xyz="0 0 0" rpy="1.5708 0 0"/>
+        <geometry>
+          <cylinder radius="0.1" length="0.05"/>
+        </geometry>
+      </collision>
+      <inertial>
+        <origin xyz="0 0 0" rpy="1.5708 0 0"/>
+        <mass value="1.0"/>
+        <inertia ixx="0.01" ixy="0.0" ixz="0.0" iyy="0.01" iyz="0.0" izz="0.01"/>
+      </inertial>
+    </link>
+    <!-- Right wheel -->
+    <link name="${prefix}right_wheel">
+      <visual>
+        <origin xyz="0 0 0" rpy="1.5708 0 0"/>
+        <geometry>
+          <cylinder radius="0.1" length="0.05"/>
+        </geometry>
+        <material name="black">
+          <color rgba="0 0 0 1"/>
+        </material>
+      </visual>
+      <collision>
+        <origin xyz="0 0 0" rpy="1.5708 0 0"/>
+        <geometry>
+          <cylinder radius="0.1" length="0.05"/>
+        </geometry>
+      </collision>
+      <inertial>
+        <origin xyz="0 0 0" rpy="1.5708 0 0"/>
+        <mass value="1.0"/>
+        <inertia ixx="0.01" ixy="0.0" ixz="0.0" iyy="0.01" iyz="0.0" izz="0.01"/>
+      </inertial>
+    </link>
+    <!-- Left wheel joint -->
+    <joint name="${prefix}left_wheel_joint" type="continuous">
+      <origin xyz="0 0.15 0" rpy="0 0 0"/>
+      <parent link="${prefix}base_link"/>
+      <child link="${prefix}left_wheel"/>
+      <axis xyz="0 1 0"/>
+    </joint>
+    <!-- Right wheel joint -->
+    <joint name="${prefix}right_wheel_joint" type="continuous">
+      <origin xyz="0 -0.15 0" rpy="0 0 0"/>
+      <parent link="${prefix}base_link"/>
+      <child link="${prefix}right_wheel"/>
+      <axis xyz="0 1 0"/>
+    </joint>
+  </xacro:macro>
   <xacro:diffbot prefix="$(arg prefix)" />
   <xacro:diffbot_ros2_control
